Commit message: upd

File: src/hexa_description/urdf/hexa_float.urdf (robot description, URDF)
Before this commit: robot floatingbase, 33 links, 32 joints
Links:
- removed link FreeFlyerRX_Link
- removed link FreeFlyerRY_Link
- removed link FreeFlyerX_Link
- removed link FreeFlyerY_Link
- removed link FreeFlyerZ_Link
- removed link base_link_2
- removed link lidar_link
- removed link rgbd_link
- added link ldlidar_base, mass 0.000010; visual mesh filename=package://hexa_description/meshes/stl/hexo_base_v1.001.stl scale=1.000000 1.000000 1.000000
Joints:
- removed joint FreeFlyerRX
- removed joint FreeFlyerRY
- removed joint FreeFlyerRZ
- removed joint FreeFlyerX
- removed joint FreeFlyerY
- removed joint FreeFlyerZ
- removed joint lidar_joint
- removed joint rgbd_joint
- joint leg1_link1_joint: parent base_link_2 -> ldlidar_base
- joint leg2_link1_joint: parent base_link_2 -> ldlidar_base
- joint leg3_link1_joint: parent base_link_2 -> ldlidar_base
- joint leg4_link1_joint: parent base_link_2 -> ldlidar_base
- joint leg5_link1_joint: parent base_link_2 -> ldlidar_base
- joint leg6_link1_joint: parent base_link_2 -> ldlidar_base
